File: EagleData/1114FN28-Kids-Shiled.brd (EAGLE design)
At the start: 86 x 53 mm, 21 parts

Commit message: Chnge TP
Parts:
- removed U$10, U$6, U$9: SIPS-2, Aruduino-Kids-Shiled:SIPC-2
- added U$8: SIPS-10, 1114FN28-Kids-Shiled:SIPS-10
- U$3: value SIPS-7 -> SIPS-5; device Aruduino-Kids-Shiled:SIPC-7 -> 1114FN28-Kids-Shiled:SIPS-5
- moved U$3 77.0 mm to (78.7, 15.2), flipped to the bottom, turned to 90 degrees
Connections:
- removed net N$26: U$1.P$16, U$6.P$1
- removed net N$27: U$1.P$15, U$6.P$2
- new net N$85: U$1.P$21, U$8.8
- new net RX: U$1.P$15, U$3.5
- new net TX: U$1.P$16, U$3.4
- net 3.3V: now also U$8.10
- net A-GND: now also U$8.9; no longer U$3.P$8
- net GND: now also U$3.2; no longer U$10.P$2, U$9.P$2
- net N$10: now also U$8.1; no longer U$3.P$1
- net N$12: now also U$8.4; no longer U$3.P$4
- net N$14: now also U$8.2; no longer U$3.P$2
- net N$15: now also U$8.3; no longer U$3.P$3
- net N$16: now also U$8.5; no longer U$3.P$5
- net N$17: now also U$8.6; no longer U$3.P$6
- net N$25: now also U$8.7; no longer U$3.P$7
- net P18: now also U$3.3; no longer U$10.P$1
- net P24: now also U$3.1; no longer U$9.P$1
Routing:
- net TX: track 0.00 -> 79.1 mm, vias 0 -> 3
- net RX: track 0.00 -> 68.0 mm, vias 0 -> 3
- net N$85: track 0.00 -> 48.1 mm, vias 0 -> 1
- net N$26: track 14.9 -> 0.00 mm
- net N$27: track 13.1 -> 0.00 mm
- net GND: track 217.7 -> 206.0 mm
- net 3.3V: track 98.3 -> 107.2 mm
- net A-GND: track 139.6 -> 136.4 mm
- net P18: track 101.1 -> 104.1 mm
- net P24: track 103.2 -> 105.9 mm
- net N$25: track 50.0 -> 48.9 mm
- net N$15: track 22.6 -> 21.9 mm
Other:
- board text added: "dp-18"
- board text added: "dp-24"
- board text added: "dp21-(3.3v In)"
- board text added: "dp7"
- board text removed: "Serial"
- board text removed: "TP3"
- board text removed: "TP4"
- board text removed: "dp18"
- board text removed: "dp24"

Commit message: Change Sch
Parts:
- moved TACTSW1 0.36 mm to (54.9, 45.4)
Connections:
- removed net N$11 (its old number): TACTSW2.3, TACTSW2.4, U$1.P$23
- net N$15: now also TACTSW2.3, TACTSW2.4
Routing:
- net N$15: track 21.9 -> 93.1 mm, vias 0 -> 2
- net N$11 (its old number): track 59.3 -> 0.00 mm
- net N$9: track 35.7 -> 31.0 mm
- net P18: track 104.1 -> 108.3 mm
- net RX: track 68.0 -> 68.2 mm, vias 3 -> 1
