File: EagleData/1114FN28-Kids-Shiled.sch (EAGLE design)
At the start: 18 parts

Commit message: Change Sch
Connections:
- removed net N$11 (its old number): TACTSW2.1, TACTSW2.3, U$1.23
- net N$15: now also TACTSW2.1, TACTSW2.3
Other:
- note added: "GND"
- note added: "dp18(PwmOut)"
- note added: "dp24(PwmOut)"
- note added: "dp7-(Analog 3.3v)"
- moved on the sheet: T-SW1, VR.1
